File: pcb_design/pcb_design.sch (KiCad schematic (older format))
At the start: 6 parts, among them U1 ATmega2560-16AU

Commit message: Damn this is cool
Parts:
- added J1: PWR, symbol Connector_Generic:Conn_01x02
- added J2: ESP8266_conn, symbol Connector_Generic:Conn_02x04_Top_Bottom
- added R3: 10K, symbol Device:R
- added R4: 20K, symbol Device:R
- added U2: LD1117S33TR_SOT223, Package_TO_SOT_SMD:SOT-223-3_TabPin2, symbol Regulator_Linear:LD1117S33TR_SOT223
- C1, C2: footprint Capacitor_SMD:C_0603_1608Metric -> Capacitor_SMD:C_0201_0603Metric
- R1, R2: footprint Resistor_SMD:R_1806_4516Metric_Pad1.57x1.80mm_HandSolder -> Resistor_SMD:R_0603_1608Metric
Connections:
- net labels added: 3_3V, 5V, ESP_EN, ESP_IO0, ESP_RST, ESP_RX, ESP_TX, RX2, TX2
- wire segments 17 -> 45
Other:
- note added: "(ESP IO2)"
- note added: "(ESP VCC)"
- note added: "Step down voltage going to ESP8266 from 5V to 3.3V \nTechnically works without, but probably better for longevity"
Changed lines of the file:
@@
 	0    1    1    0
 $EndComp
+Wire Wire Line
+	2000 1250 2600 1250
+Wire Wire Line
+	2600 1300 2600 1250
+Wire Wire Line
+	2600 1500 2600 1550
+Wire Wire Line
+	2000 1250 1850 1250
+Connection ~ 2000 1250
+Wire Wire Line
+	2000 1550 1850 1550
+Connection ~ 2000 1550
+Wire Wire Line
+	1650 1250 1650 1400
+Wire Wire Line
+	1650 1400 1600 1400
+Connection ~ 1650 1400
+Wire Wire Line
+	1650 1400 1650 1550
+Text Label 1600 1400 2    50   ~ 0
+GND
+$Comp
+L Device:R R1
+U 1 1 60717ACE
+P 1300 1400
+F 0 "R1" H 1350 1350 50  0000 L CNN
+F 1 "1M" V 1300 1350 50  0000 L CNN
+F 2 "Resistor_SMD:R_0603_1608Metric" V 1230 1400 50  0001 C CNN
+F 3 "~" H 1300 1400 50  0001 C CNN
+	1    1300 1400
+	1    0    0    -1
+$EndComp
+Wire Wire Line
+	2000 1550 2000 1700
+Wire Wire Line
+	2000 1700 1300 1700
+Wire Wire Line
+	1300 1700 1300 1550
+Wire Wire Line
+	2000 1250 2000 1100
+Wire Wire Line
+	2000 1100 1300 1100
+Wire Wire Line
+	1300 1100 1300 1250
+$Comp
+L Device:R R2
+U 1 1 6072866C
+P 2350 1550
+F 0 "R2" V 2450 1450 50  0000 C CNN
+F 1 "27" V 2450 1550 50  0000 C CNN
+F 2 "Resistor_SMD:R_0603_1608Metric" V 2280 1550 50  0001 C CNN
+F 3 "~" H 2350 1550 50  0001 C CNN
+	1    2350 1550
+	0    1    1    0
+$EndComp
+Wire Wire Line
+	2000 1550 2200 1550
+Wire Wire Line
+	2500 1550 2600 1550
+Wire Wire Line
+	2600 1100 2350 1100
+Text Label 2350 1100 0    50   ~ 0
+RST
+Text Label 3400 6600 0    50   ~ 0
+GND
+$Comp
+L Device:C_Small C1
+U 1 1 6071040A
+P 1750 1250
+F 0 "C1" V 1550 1250 50  0000 C CNN
+F 1 "22pF" V 1650 1250 50  0000 C CNN
+F 2 "Capacitor_SMD:C_0201_0603Metric" H 1750 1250 50  0001 C CNN
+F 3 "~" H 1750 1250 50  0001 C CNN
+	1    1750 1250
+	0    1    1    0
+$EndComp
+$Comp
+L Device:C_Small C2
+U 1 1 60710D71
+P 1750 1550
+F 0 "C2" V 1950 1550 50  0000 C CNN
+F 1 "22pF" V 1850 1550 50  0000 C CNN
+F 2 "Capacitor_SMD:C_0201_0603Metric" H 1750 1550 50  0001 C CNN
+F 3 "~" H 1750 1550 50  0001 C CNN
+	1    1750 1550
+	0    1    1    0
+$EndComp
+Wire Wire Line
+	3400 800  3400 650
+Wire Wire Line
+	3500 800  3500 650
+Wire Wire Line
+	3500 650  3400 650
+Wire Wire Line
+	3500 650  3600 650
+Connection ~ 3500 650
+Text Label 3600 650  0    50   ~ 0
+5V
+$Comp
+L Connector_Generic:Conn_01x02 J1
+U 1 1 606DA8B0
+P 5700 1100
+F 0 "J1" H 5780 1092 50  0000 L CNN
+F 1 "PWR" H 5780 1001 50  0000 L CNN
+F 2 "" H 5700 1100 50  0001 C CNN
+F 3 "~" H 5700 1100 50  0001 C CNN
+	1    5700 1100
+	1    0    0    -1
+$EndComp
+Wire Wire Line
+	5500 1100 5400 1100
+Wire Wire Line
+	5500 1200 5400 1200
+Text Label 5400 1100 2    50   ~ 0
+5V
+Text Label 5400 1200 2    50   ~ 0
+GND
+$Comp
+L Regulator_Linear:LD1117S33TR_SOT223 U2
+U 1 1 606F0FA3
+P 5550 1750
+F 0 "U2" H 5550 1992 50  0000 C CNN
+F 1 "LD1117S33TR_SOT223" H 5550 1901 50  0000 C CNN
+F 2 "Package_TO_SOT_SMD:SOT-223-3_TabPin2" H 5550 1950 50  0001 C CNN
+F 3 "http://www.st.com/st-web-ui/static/active/en/resource/technical/document/datasheet/CD00000544.pdf" H 5650 1500 50  0001 C CNN
+	1    5550 1750
+	1    0    0    -1
+$EndComp
+Wire Wire Line
+	5550 2050 5550 2250
+Wire Wire Line
+	5850 1750 6000 1750
+Wire Wire Line
+	5250 1750 5050 1750
+Text Label 6000 1750 0    50   ~ 0
+3_3V
+Text Label 5050 1750 0    50   ~ 0
+5V
+Text Label 5550 2250 0    50   ~ 0
+GND
+$Comp
+L Connector_Generic:Conn_02x04_Top_Bottom J2
+U 1 1 60700AF7
+P 5750 3400
+F 0 "J2" H 5800 3717 50  0000 C CNN
+F 1 "ESP8266_conn" H 5800 3626 50  0000 C CNN
+F 2 "" H 5750 3400 50  0001 C CNN
+F 3 "~" H 5750 3400 50  0001 C CNN
+	1    5750 3400
+	1    0    0    -1
+$EndComp
+Wire Wire Line
+	6050 3300 6200 3300
+Wire Wire Line
+	6050 3400 6200 3400
+Wire Wire Line
+	6050 3500 6200 3500
+Wire Wire Line
+	6050 3600 6200 3600
+Wire Wire Line
+	5550 3300 5400 3300
+Wire Wire Line
+	5550 3400 5400 3400
+Wire Wire Line
+	5550 3500 5400 3500
+Wire Wire Line
+	5550 3600 5400 3600
+Text Label 5400 3300 2    50   ~ 0
+ESP_RX
+Text Label 5400 3500 2    50   ~ 0
+3_3V
+Text Label 5400 3600 2    50   ~ 0
+GND
+Text Label 6200 3600 0    50   ~ 0
+ESP_TX
+Text Label 6200 3300 0    50   ~ 0
+3_3V
+Text Notes 6400 3300 0    50   ~ 0
+(ESP VCC)
+Text Notes 4800 3500 0    50   ~ 0
+(ESP IO2)
+Text Label 6200 3400 0    50   ~ 0
+ESP_RST
+Text Label 5400 3400 2    50   ~ 0
+ESP_IO0
+Wire Wire Line
+	5500 3800 5750 3800
+Wire Wire Line
+	5500 3900 5750 3900
+Text Label 5500 3800 2    50   ~ 0
+ESP_IO0
+Text Label 5750 3800 0    50   ~ 0
+3_3V
+Text Label 5750 3900 0    50   ~ 0
+3_3V
+Text Label 5500 3900 2    50   ~ 0
+ESP_RST
+Text Label 6200 3500 0    50   ~ 0
+ESP_EN
+Wire Wire Line
+	5500 4000 5750 4000
+Text Label 5750 4000 0    50   ~ 0
+3_3V
+Text Label 5500 4000 2    50   ~ 0
+ESP_EN
+$Comp
+L Device:R R3
+U 1 1 60719578
+P 5400 4600
+F 0 "R3" V 5193 4600 50  0000 C CNN
+F 1 "10K" V 5284 4600 50  0000 C CNN
+F 2 "" V 5330 4600 50  0001 C CNN
+F 3 "~" H 5400 4600 50  0001 C CNN
+	1    5400 4600
+	0    1    1    0
+$EndComp
+$Comp
+L Device:R R4
+U 1 1 60719C63
+P 5900 4600
+F 0 "R4" V 5693 4600 50  0000 C CNN
+F 1 "20K" V 5784 4600 50  0000 C CNN
+F 2 "" V 5830 4600 50  0001 C CNN
+F 3 "~" H 5900 4600 50  0001 C CNN
+	1    5900 4600
+	0    1    1    0
+$EndComp
+Wire Wire Line
+	5100 4600 5250 4600
+Wire Wire Line
+	6050 4600 6200 4600
+Text Label 6200 4600 0    50   ~ 0
+GND
+Text Label 5100 4600 2    50   ~ 0
+TX2
+Text Label 5650 4800 2    50   ~ 0
+ESP_RX
+Wire Wire Line
+	5550 4600 5650 4600
+Wire Wire Line
+	5650 4600 5650 4800
+Connection ~ 5650 4600
+Wire Wire Line
+	5650 4600 5750 4600
 $Comp
 L Atmega:ATmega2560-16AU U1
@@
 $EndComp
 Wire Wire Line
-	2000 1250 2600 1250
-Wire Wire Line
-	2600 1300 2600 1250
-Wire Wire Line
-	2600 1500 2600 1550
-Wire Wire Line
-	2000 1250 1850 1250
-Connection ~ 2000 1250
-Wire Wire Line
-	2000 1550 1850 1550
-Connection ~ 2000 1550
-Wire Wire Line
-	1650 1250 1650 1400
-Wire Wire Line
-	1650 1400 1600 1400
-Connection ~ 1650 1400
-Wire Wire Line
-	1650 1400 1650 1550
-Text Label 1600 1400 2    50   ~ 0
-GND
-$Comp
-L Device:R R1
-U 1 1 60717ACE
-P 1300 1400
-F 0 "R1" H 1350 1350 50  0000 L CNN
-F 1 "1M" V 1300 1350 50  0000 L CNN
-F 2 "Resistor_SMD:R_1806_4516Metric_Pad1.57x1.80mm_HandSolder" V 1230 1400 50  0001 C CNN
-F 3 "~" H 1300 1400 50  0001 C CNN
-	1    1300 1400
-	1    0    0    -1
-$EndComp
-Wire Wire Line
-	2000 1550 2000 1700
-Wire Wire Line
-	2000 1700 1300 1700
-Wire Wire Line
-	1300 1700 1300 1550
-Wire Wire Line
-	2000 1250 2000 1100
-Wire Wire Line
-	2000 1100 1300 1100
-Wire Wire Line
-	1300 1100 1300 1250
-$Comp
-L Device:R R2
-U 1 1 6072866C
-P 2350 1550
-F 0 "R2" V 2450 1450 50  0000 C CNN
-F 1 "27" V 2450 1550 50  0000 C CNN
-F 2 "Resistor_SMD:R_1806_4516Metric_Pad1.57x1.80mm_HandSolder" V 2280 1550 50  0001 C CNN
-F 3 "~" H 2350 1550 50  0001 C CNN
-	1    2350 1550
-	0    1    1    0
-$EndComp
-Wire Wire Line
-	2000 1550 2200 1550
-Wire Wire Line
-	2500 1550 2600 1550
-Wire Wire Line
-	2600 1100 2350 1100
-Text Label 2350 1100 0    50   ~ 0
-RST
-Text Label 3400 6600 0    50   ~ 0
-GND
-$Comp
-L Device:C_Small C1
-U 1 1 6071040A
-P 1750 1250
-F 0 "C1" V 1550 1250 50  0000 C CNN
-F 1 "22pF" V 1650 1250 50  0000 C CNN
-F 2 "Capacitor_SMD:C_0603_1608Metric" H 1750 1250 50  0001 C CNN
-F 3 "~" H 1750 1250 50  0001 C CNN
-	1    1750 1250
-	0    1    1    0
-$EndComp
-$Comp
-L Device:C_Small C2
-U 1 1 60710D71
-P 1750 1550
-F 0 "C2" V 1950 1550 50  0000 C CNN
-F 1 "22pF" V 1850 1550 50  0000 C CNN
-F 2 "Capacitor_SMD:C_0603_1608Metric" H 1750 1550 50  0001 C CNN
-F 3 "~" H 1750 1550 50  0001 C CNN
-	1    1750 1550
-	0    1    1    0
-$EndComp
+	2600 4700 2400 4700
+Wire Wire Line
+	2600 4800 2400 4800
+Text Label 2400 4700 2    50   ~ 0
+RX2
+Text Label 2400 4800 2    50   ~ 0
+TX2
+Wire Wire Line
+	5500 4100 5750 4100
+Text Label 5500 4100 2    50   ~ 0
+ESP_TX
+Text Label 5750 4100 0    50   ~ 0
+RX2
+Text Notes 5800 4850 0    50   ~ 0
+Step down voltage going to ESP8266 from 5V to 3.3V \nTechnically works without, but probably better for longevity
 $EndSCHEMATC

Commit message: Add small thingoes
Parts:
- added C? (x2): 22pF, Capacitor_SMD:C_0201_0603Metric, symbol Device:C_Small
- added C? (x3): 100nF, symbol Device:C
- added Clk?: 16Mhz, Crystal:Crystal_HC52-8mm_Vertical, symbol Device:Crystal
- added R?: 1M, Resistor_SMD:R_0603_1608Metric, symbol Device:R
- added R?: 27, Resistor_SMD:R_0603_1608Metric, symbol Device:R
- added U?: ATmega8U2-AU, Package_QFP:TQFP-32_7x7mm_P0.8mm, symbol MCU_Microchip_ATmega:ATmega8U2-AU
- U1: symbol Atmega:ATmega2560-16AU -> pcb_design-rescue:ATmega2560-16AU-Atmega
Connections:
- net labels added: +3.3V, +5V
- net labels removed: 3_3V, 5V
- wire segments 45 -> 68

Commit message: Move and stuff
Parts:
- removed C? (x2): 22pF, Capacitor_SMD:C_0201_0603Metric, symbol Device:C_Small
- removed Clk?: 16Mhz, Crystal:Crystal_HC52-8mm_Vertical, symbol Device:Crystal
- removed R?: 1M, Resistor_SMD:R_0603_1608Metric, symbol Device:R
- removed R?: 27, Resistor_SMD:R_0603_1608Metric, symbol Device:R
- removed U?: ATmega8U2-AU, Package_QFP:TQFP-32_7x7mm_P0.8mm, symbol MCU_Microchip_ATmega:ATmega8U2-AU
- U1: symbol pcb_design-rescue:ATmega2560-16AU-Atmega -> pcb_design-rescue:ATmega2560-16AU-Atmega-pcb_design-rescue
- gave numbers to parts that had none: 3
Connections:
- wire segments 68 -> 51
Changed lines of the file:
@@
 $Descr A4 11693 8268
 encoding utf-8
-Sheet 1 1
+Sheet 1 2
 Title ""
 Date ""
@@
 	5650 4600 5750 4600
 $Comp
-L pcb_design-rescue:ATmega2560-16AU-Atmega U1
+L pcb_design-rescue:ATmega2560-16AU-Atmega-pcb_design-rescue U1
 U 1 1 606E4022
 P 3400 3700
@@
 Step down voltage going to ESP8266 from 5V to 3.3V \nTechnically works without, but probably better for longevity
 $Comp
-L MCU_Microchip_ATmega:ATmega8U2-AU U?
-U 1 1 606FBABA
-P 9550 2550
-F 0 "U?" H 9550 1061 50  0000 C CNN
-F 1 "ATmega8U2-AU" H 9550 970 50  0000 C CNN
-F 2 "Package_QFP:TQFP-32_7x7mm_P0.8mm" H 9550 2550 50  0001 C CIN
-F 3 "http://ww1.microchip.com/downloads/en/DeviceDoc/doc7799.pdf" H 9550 2550 50  0001 C CNN
-	1    9550 2550
-	1    0    0    -1
-$EndComp
-$Comp
-L Device:Crystal Clk?
-U 1 1 60708925
-P 8200 1750
-F 0 "Clk?" V 8154 1881 50  0000 L CNN
-F 1 "16Mhz" V 8245 1881 50  0000 L CNN
-F 2 "Crystal:Crystal_HC52-8mm_Vertical" H 8200 1750 50  0001 C CNN
-F 3 "~" H 8200 1750 50  0001 C CNN
-	1    8200 1750
-	0    1    1    0
-$EndComp
-Wire Wire Line
-	8200 1600 8800 1600
-Wire Wire Line
-	8200 1600 8050 1600
-Connection ~ 8200 1600
-Wire Wire Line
-	8200 1900 8050 1900
-Connection ~ 8200 1900
-Wire Wire Line
-	7850 1600 7850 1750
-Connection ~ 7850 1750
-Wire Wire Line
-	7850 1750 7850 1900
-$Comp
-L Device:R R?
-U 1 1 60708935
-P 7500 1750
-F 0 "R?" H 7550 1700 50  0000 L CNN
-F 1 "1M" V 7500 1700 50  0000 L CNN
-F 2 "Resistor_SMD:R_0603_1608Metric" V 7430 1750 50  0001 C CNN
-F 3 "~" H 7500 1750 50  0001 C CNN
-	1    7500 1750
-	1    0    0    -1
-$EndComp
-Wire Wire Line
-	8200 1900 8200 2050
-Wire Wire Line
-	8200 2050 7500 2050
-Wire Wire Line
-	7500 2050 7500 1900
-Wire Wire Line
-	8200 1600 8200 1450
-Wire Wire Line
-	8200 1450 7500 1450
-Wire Wire Line
-	7500 1450 7500 1600
-$Comp
-L Device:R R?
-U 1 1 60708941
-P 8550 1900
-F 0 "R?" V 8650 1800 50  0000 C CNN
-F 1 "27" V 8650 1900 50  0000 C CNN
-F 2 "Resistor_SMD:R_0603_1608Metric" V 8480 1900 50  0001 C CNN
-F 3 "~" H 8550 1900 50  0001 C CNN
-	1    8550 1900
-	0    1    1    0
-$EndComp
-Wire Wire Line
-	8200 1900 8400 1900
-Wire Wire Line
-	8700 1900 8800 1900
-$Comp
-L Device:C_Small C?
-U 1 1 6070894B
-P 7950 1600
-F 0 "C?" V 7750 1600 50  0000 C CNN
-F 1 "22pF" V 7850 1600 50  0000 C CNN
-F 2 "Capacitor_SMD:C_0201_0603Metric" H 7950 1600 50  0001 C CNN
-F 3 "~" H 7950 1600 50  0001 C CNN
-	1    7950 1600
-	0    1    1    0
-$EndComp
-$Comp
-L Device:C_Small C?
-U 1 1 60708951
-P 7950 1900
-F 0 "C?" V 8150 1900 50  0000 C CNN
-F 1 "22pF" V 8050 1900 50  0000 C CNN
-F 2 "Capacitor_SMD:C_0201_0603Metric" H 7950 1900 50  0001 C CNN
-F 3 "~" H 7950 1900 50  0001 C CNN
-	1    7950 1900
-	0    1    1    0
-$EndComp
-$Comp
-L power:+5V #PWR?
+L power:+5V #PWR0101
 U 1 1 6071B869
 P 5400 1100
-F 0 "#PWR?" H 5400 950 50  0001 C CNN
+F 0 "#PWR0101" H 5400 950 50  0001 C CNN
 F 1 "+5V" V 5415 1228 50  0000 L CNN
 F 2 "" H 5400 1100 50  0001 C CNN
@@
 $EndComp
 $Comp
-L power:GND #PWR?
+L power:GND #PWR0102
 U 1 1 6071E840
 P 5400 1200
-F 0 "#PWR?" H 5400 950 50  0001 C CNN
+F 0 "#PWR0102" H 5400 950 50  0001 C CNN
 F 1 "GND" V 5405 1072 50  0000 R CNN
 F 2 "" H 5400 1200 50  0001 C CNN
@@
 $EndComp
 $Comp
-L power:GND #PWR?
+L power:GND #PWR0103
 U 1 1 6072142C
 P 5550 2250
-F 0 "#PWR?" H 5550 2000 50  0001 C CNN
+F 0 "#PWR0103" H 5550 2000 50  0001 C CNN
 F 1 "GND" H 5555 2077 50  0000 C CNN
 F 2 "" H 5550 2250 50  0001 C CNN
@@
 $EndComp
 $Comp
-L power:GND #PWR?
-U 1 1 607265F7
-P 7700 1750
-F 0 "#PWR?" H 7700 1500 50  0001 C CNN
-F 1 "GND" H 7705 1577 50  0000 C CNN
-F 2 "" H 7700 1750 50  0001 C CNN
-F 3 "" H 7700 1750 50  0001 C CNN
-	1    7700 1750
-	1    0    0    -1
-$EndComp
-Wire Wire Line
-	7700 1750 7850 1750
-$Comp
-L power:+3.3V #PWR?
+L power:+3.3V #PWR0105
 U 1 1 60732717
 P 6000 1750
-F 0 "#PWR?" H 6000 1600 50  0001 C CNN
+F 0 "#PWR0105" H 6000 1600 50  0001 C CNN
 F 1 "+3.3V" V 6015 1878 50  0000 L CNN
 F 2 "" H 6000 1750 50  0001 C CNN
@@
 $EndComp
 $Comp
-L power:+5V #PWR?
+L power:+5V #PWR0106
 U 1 1 607339F0
 P 5050 1750
-F 0 "#PWR?" H 5050 1600 50  0001 C CNN
+F 0 "#PWR0106" H 5050 1600 50  0001 C CNN
 F 1 "+5V" V 5065 1878 50  0000 L CNN
 F 2 "" H 5050 1750 50  0001 C CNN
@@
 $EndComp
 $Comp
-L power:+3.3V #PWR?
+L power:+3.3V #PWR0107
 U 1 1 60736BC4
 P 5750 3800
-F 0 "#PWR?" H 5750 3650 50  0001 C CNN
+F 0 "#PWR0107" H 5750 3650 50  0001 C CNN
 F 1 "+3.3V" V 5765 3928 50  0000 L CNN
 F 2 "" H 5750 3800 50  0001 C CNN
@@
 $EndComp
 $Comp
-L power:+3.3V #PWR?
+L power:+3.3V #PWR0108
 U 1 1 60737357
 P 5750 3900
-F 0 "#PWR?" H 5750 3750 50  0001 C CNN
+F 0 "#PWR0108" H 5750 3750 50  0001 C CNN
 F 1 "+3.3V" V 5765 4028 50  0000 L CNN
 F 2 "" H 5750 3900 50  0001 C CNN
@@
 $EndComp
 $Comp
-L power:+3.3V #PWR?
+L power:+3.3V #PWR0109
 U 1 1 60737C45
 P 5750 4000
-F 0 "#PWR?" H 5750 3850 50  0001 C CNN
+F 0 "#PWR0109" H 5750 3850 50  0001 C CNN
 F 1 "+3.3V" V 5765 4128 50  0000 L CNN
 F 2 "" H 5750 4000 50  0001 C CNN
@@
 $EndComp
 $Comp
-L power:GND #PWR?
+L power:GND #PWR0110
 U 1 1 607393F6
 P 6200 4600
-F 0 "#PWR?" H 6200 4350 50  0001 C CNN
+F 0 "#PWR0110" H 6200 4350 50  0001 C CNN
 F 1 "GND" V 6205 4472 50  0000 R CNN
 F 2 "" H 6200 4600 50  0001 C CNN
@@
 $EndComp
 $Comp
-L power:GND #PWR?
+L power:GND #PWR0111
 U 1 1 6074E330
 P 3400 6600
-F 0 "#PWR?" H 3400 6350 50  0001 C CNN
+F 0 "#PWR0111" H 3400 6350 50  0001 C CNN
 F 1 "GND" V 3405 6472 50  0000 R CNN
 F 2 "" H 3400 6600 50  0001 C CNN
@@
 $EndComp
 $Comp
-L power:+3.3V #PWR?
+L power:+3.3V #PWR0112
 U 1 1 6075286B
 P 5400 3500
-F 0 "#PWR?" H 5400 3350 50  0001 C CNN
+F 0 "#PWR0112" H 5400 3350 50  0001 C CNN
 F 1 "+3.3V" V 5415 3628 50  0000 L CNN
 F 2 "" H 5400 3500 50  0001 C CNN
@@
 $EndComp
 $Comp
-L power:+3.3V #PWR?
+L power:+3.3V #PWR0113
 U 1 1 60758694
 P 6200 3300
-F 0 "#PWR?" H 6200 3150 50  0001 C CNN
+F 0 "#PWR0113" H 6200 3150 50  0001 C CNN
 F 1 "+3.3V" H 6215 3473 50  0000 C CNN
 F 2 "" H 6200 3300 50  0001 C CNN
@@
 $EndComp
 $Comp
-L power:GND #PWR?
+L power:GND #PWR0114
 U 1 1 6075C443
 P 5400 3600
-F 0 "#PWR?" H 5400 3350 50  0001 C CNN
+F 0 "#PWR0114" H 5400 3350 50  0001 C CNN
 F 1 "GND" V 5405 3472 50  0000 R CNN
 F 2 "" H 5400 3600 50  0001 C CNN
@@
 $EndComp
 $Comp
-L power:+5V #PWR?
-U 1 1 60765D4B
-P 9550 1050
-F 0 "#PWR?" H 9550 900 50  0001 C CNN
-F 1 "+5V" H 9565 1223 50  0000 C CNN
-F 2 "" H 9550 1050 50  0001 C CNN
-F 3 "" H 9550 1050 50  0001 C CNN
-	1    9550 1050
-	1    0    0    -1
-$EndComp
-Wire Wire Line
-	9550 1050 9550 1150
-Wire Wire Line
-	9550 1050 9650 1050
-Wire Wire Line
-	9650 1050 9650 1150
-Connection ~ 9550 1050
-$Comp
-L power:GND #PWR?
-U 1 1 60769128
-P 9550 3950
-F 0 "#PWR?" H 9550 3700 50  0001 C CNN
-F 1 "GND" V 9555 3822 50  0000 R CNN
-F 2 "" H 9550 3950 50  0001 C CNN
-F 3 "" H 9550 3950 50  0001 C CNN
-	1    9550 3950
-	0    -1   -1   0
-$EndComp
-$Comp
-L power:GND #PWR?
+L power:GND #PWR0117
 U 1 1 60775CB5
 P 1500 1400
-F 0 "#PWR?" H 1500 1150 50  0001 C CNN
+F 0 "#PWR0117" H 1500 1150 50  0001 C CNN
 F 1 "GND" H 1505 1227 50  0000 C CNN
 F 2 "" H 1500 1400 50  0001 C CNN
@@
 Connection ~ 3500 500
 $Comp
-L Device:C C?
+L Device:C C3
 U 1 1 60784AD5
 P 3700 650
-F 0 "C?" H 3815 696 50  0000 L CNN
+F 0 "C3" H 3815 696 50  0000 L CNN
 F 1 "100nF" H 3815 605 50  0000 L CNN
 F 2 "" H 3738 500 50  0001 C CNN
@@
 Connection ~ 3700 500
 $Comp
-L Device:C C?
+L Device:C C4
 U 1 1 607854A5
 P 4150 650
-F 0 "C?" H 4265 696 50  0000 L CNN
+F 0 "C4" H 4265 696 50  0000 L CNN
 F 1 "100nF" H 4265 605 50  0000 L CNN
 F 2 "" H 4188 500 50  0001 C CNN
@@
 $EndComp
 $Comp
-L Device:C C?
+L Device:C C5
 U 1 1 60785959
 P 4600 650
-F 0 "C?" H 4715 696 50  0000 L CNN
+F 0 "C5" H 4715 696 50  0000 L CNN
 F 1 "100nF" H 4715 605 50  0000 L CNN
 F 2 "" H 4638 500 50  0001 C CNN
@@
 Connection ~ 4600 500
 $Comp
-L power:+5V #PWR?
+L power:+5V #PWR0118
 U 1 1 60788B7F
 P 4750 500
-F 0 "#PWR?" H 4750 350 50  0001 C CNN
+F 0 "#PWR0118" H 4750 350 50  0001 C CNN
 F 1 "+5V" V 4765 628 50  0000 L CNN
 F 2 "" H 4750 500 50  0001 C CNN
@@
 	4600 800  4750 800
 $Comp
-L power:GND #PWR?
+L power:GND #PWR0119
 U 1 1 6078AD05
 P 4750 800
-F 0 "#PWR?" H 4750 550 50  0001 C CNN
+F 0 "#PWR0119" H 4750 550 50  0001 C CNN
 F 1 "GND" V 4755 672 50  0000 R CNN
 F 2 "" H 4750 800 50  0001 C CNN
@@
 Wire Wire Line
 	4150 800  4600 800
+$Sheet
+S 8900 4650 1200 1300
+U 606EB0A7
+F0 "atmega8u2" 50
+F1 "atmega8u2.sch" 50
+$EndSheet
 $EndSCHEMATC

Commit message: Add ISP header and bit more of USB thingo
Parts:
- added J?: ISP, symbol Connector_Generic:Conn_02x03_Counter_Clockwise
Connections:
- net labels added: MISO, MOSI, PRGM_RX, PRGM_TX, SCK
- wire segments 51 -> 65
Changed lines of the file:
@@
 F0 "atmega8u2" 50
 F1 "atmega8u2.sch" 50
+F2 "PRGM_RX" I L 8900 5700 50
+F3 "PRGM_TX" I L 8900 5800 50
+F4 "PRGM_RST" I L 8900 5600 50
 $EndSheet
+Wire Wire Line
+	4200 4700 4350 4700
+Wire Wire Line
+	4200 4800 4350 4800
+Wire Wire Line
+	8900 5700 8750 5700
+Wire Wire Line
+	8900 5800 8750 5800
+Text Label 8750 5700 2    50   ~ 0
+PRGM_RX
+Text Label 8750 5800 2    50   ~ 0
+PRGM_TX
+Text Label 4350 4700 0    50   ~ 0
+PRGM_RX
+Text Label 4350 4800 0    50   ~ 0
+PRGM_TX
+$Comp
+L Connector_Generic:Conn_02x03_Counter_Clockwise J?
+U 1 1 6071B139
+P 7500 1150
+F 0 "J?" H 7550 1467 50  0000 C CNN
+F 1 "ISP" H 7550 1376 50  0000 C CNN
+F 2 "" H 7500 1150 50  0001 C CNN
+F 3 "~" H 7500 1150 50  0001 C CNN
+	1    7500 1150
+	1    0    0    -1
+$EndComp
+Text Label 4350 2300 0    50   ~ 0
+MISO
+Text Label 4350 2100 0    50   ~ 0
+SCK
+Text Label 4350 2200 0    50   ~ 0
+MOSI
+Wire Wire Line
+	4350 2100 4200 2100
+Wire Wire Line
+	4200 2200 4350 2200
+Wire Wire Line
+	4350 2300 4200 2300
+Text Label 7150 1050 2    50   ~ 0
+MISO
+Text Label 7150 1150 2    50   ~ 0
+SCK
+Text Label 7150 1250 2    50   ~ 0
+RST
+Text Label 7950 1150 0    50   ~ 0
+MOSI
+$Comp
+L power:GND #PWR?
+U 1 1 6072BCF1
+P 7950 1250
+F 0 "#PWR?" H 7950 1000 50  0001 C CNN
+F 1 "GND" H 7955 1077 50  0000 C CNN
+F 2 "" H 7950 1250 50  0001 C CNN
+F 3 "" H 7950 1250 50  0001 C CNN
+	1    7950 1250
+	1    0    0    -1
+$EndComp
+$Comp
+L power:+5V #PWR?
+U 1 1 6072C21C
+P 7950 1050
+F 0 "#PWR?" H 7950 900 50  0001 C CNN
+F 1 "+5V" H 7965 1223 50  0000 C CNN
+F 2 "" H 7950 1050 50  0001 C CNN
+F 3 "" H 7950 1050 50  0001 C CNN
+	1    7950 1050
+	1    0    0    -1
+$EndComp
+Wire Wire Line
+	7800 1250 7950 1250
+Wire Wire Line
+	7950 1150 7800 1150
+Wire Wire Line
+	7950 1050 7800 1050
+Wire Wire Line
+	7150 1050 7300 1050
+Wire Wire Line
+	7150 1150 7300 1150
+Wire Wire Line
+	7300 1250 7150 1250
+Wire Wire Line
+	8900 5600 8750 5600
+Text Label 8750 5600 2    50   ~ 0
+RST
 $EndSCHEMATC

Commit message: Move around
Parts:
- C1, C2: symbol Device:C_Small -> pcb_design-rescue:C_Small-Device
- C3, C4, C5: symbol Device:C -> pcb_design-rescue:C-Device
- Clk1: symbol Device:Crystal -> pcb_design-rescue:Crystal-Device
- J1: symbol Connector_Generic:Conn_01x02 -> pcb_design-rescue:Conn_01x02-Connector_Generic
- J2: symbol Connector_Generic:Conn_02x04_Top_Bottom -> pcb_design-rescue:Conn_02x04_Top_Bottom-Connector_Generic
- J?: symbol Connector_Generic:Conn_02x03_Counter_Clockwise -> pcb_design-rescue:Conn_02x03_Counter_Clockwise-Connector_Generic
- R1, R2, R3, R4: symbol Device:R -> pcb_design-rescue:R-Device
- U2: symbol Regulator_Linear:LD1117S33TR_SOT223 -> pcb_design-rescue:LD1117S33TR_SOT223-Regulator_Linear
Connections:
- wire segments 65 -> 63
Other:
- moved on the sheet: R1, R2, U1
