File: pcb_design/pcb_design.sch (KiCad schematic (older format))
At the start: 15 parts, among them J1 PWR, J2 ESP8266_conn, U1 ATmega2560-16AU, U2 LD1117S33TR_SOT223

Commit message: Make PCB design
Parts:
- removed J2: ESP8266_conn, symbol pcb_design-rescue:Conn_02x04_Top_Bottom-Connector_Generic
- removed J?: ISP, symbol pcb_design-rescue:Conn_02x03_Counter_Clockwise-Connector_Generic
- added D1: LED, LED_SMD:LED_0201_0603Metric, symbol Device:LED
- added D2: LED_PWR, LED_SMD:LED_0201_0603Metric, symbol Device:LED
- added J10: PD, Connector_PinHeader_2.54mm:PinHeader_1x08_P2.54mm_Vertical, symbol Connector_Generic:Conn_01x08
- added J11: PE, Connector_PinHeader_2.54mm:PinHeader_1x08_P2.54mm_Vertical, symbol Connector_Generic:Conn_01x08
- added J12: PF, Connector_PinHeader_2.54mm:PinHeader_1x08_P2.54mm_Vertical, symbol Connector_Generic:Conn_01x08
- added J13: ICSP, Connector_PinHeader_2.54mm:PinHeader_2x03_P2.54mm_Vertical, symbol Connector_Generic:Conn_02x03_Odd_Even
- added J14: PWR_OUT, Connector_PinHeader_2.54mm:PinHeader_1x02_P2.54mm_Vertical, symbol pcb_design-rescue:Conn_01x02-Connector_Generic
- added J2: ESP8266_CONN, Connector_PinHeader_2.54mm:PinHeader_2x04_P2.54mm_Vertical, symbol Connector_Generic:Conn_02x04_Odd_Even
- added J3: PL, Connector_PinHeader_2.54mm:PinHeader_1x08_P2.54mm_Vertical, symbol Connector_Generic:Conn_01x08
- added J4: PK, Connector_PinHeader_2.54mm:PinHeader_1x08_P2.54mm_Vertical, symbol Connector_Generic:Conn_01x08
- added J5: PJ, Connector_PinHeader_2.54mm:PinHeader_1x08_P2.54mm_Vertical, symbol Connector_Generic:Conn_01x08
- added J6: PH, Connector_PinHeader_2.54mm:PinHeader_1x05_P2.54mm_Vertical, symbol Connector_Generic:Conn_01x05
- added J7: PA, Connector_PinHeader_2.54mm:PinHeader_1x08_P2.54mm_Vertical, symbol Connector_Generic:Conn_01x08
- added J8: PB, Connector_PinHeader_2.54mm:PinHeader_1x08_P2.54mm_Vertical, symbol Connector_Generic:Conn_01x08
- added J9: PC, Connector_PinHeader_2.54mm:PinHeader_1x08_P2.54mm_Vertical, symbol Connector_Generic:Conn_01x08
- added R7, R9: 1K, Resistor_SMD:R_0201_0603Metric, symbol Device:R
- added R8: 10K, Resistor_SMD:R_0201_0603Metric, symbol Device:R
- added SW1: SW_Push, Button_Switch_SMD:SW_SPST_B3U-1000P, symbol Switch:SW_Push
- C3, C4, C5: footprint (none) -> Capacitor_SMD:C_0201_0603Metric
- J1: value PWR -> PWR_IN; footprint (none) -> Connector_PinHeader_2.54mm:PinHeader_1x02_P2.54mm_Vertical
- R1, R2: footprint Resistor_SMD:R_0603_1608Metric -> Resistor_SMD:R_0201_0603Metric
- R3, R4: footprint (none) -> Resistor_SMD:R_0201_0603Metric
Connections:
- net +3V3: now also J2.2 (Pin_2), J2.3 (Pin_3), J2.4 (Pin_4), J2.5 (Pin_5), J2.6 (Pin_6)
- net +5V: now also U2.3 (VI), J13.2 (Pin_2), J14.2 (Pin_2), R8.1, R9.2
- net ESP_RX: now also R3.2, R4.1, J2.1 (Pin_1); no longer R3.1, R4.2
- net ESP_TX: now also J2.8 (Pin_8)
- net GND: now also R4.2, D1.1 (K), D2.1 (K), J13.6 (Pin_6), J14.1 (Pin_1), J2.7 (Pin_7), SW1.2; no longer R4.1
- net MISO: now also J13.1 (Pin_1), J8.4 (Pin_4)
- net MOSI: now also J13.4 (Pin_4), J8.3 (Pin_3)
- net PRGM_RX: now also U1.2 (PE0), J11.1 (Pin_1)
- net PRGM_TX: now also U1.3 (PE1), J11.2 (Pin_2)
- net RST: now also J13.5 (Pin_5), R8.2, SW1.1
- net SCK: now also J13.3 (Pin_3), J8.2 (Pin_2)
- net TX2: now also R3.1
- net at U1.1 (PG5): now also R7.2
- net at U1.14 (PH2): now also J6.1 (Pin_1)
- net at U1.15 (PH3): now also J6.2 (Pin_2)
- net at U1.16 (PH4): now also J6.3 (Pin_3)
- net at U1.17 (PH5): now also J6.4 (Pin_4)
- net at U1.18 (PH6): now also J6.5 (Pin_5)
- net at U1.19 (PB0): now also J8.1 (Pin_1)
- net at U1.23 (PB4): now also J8.5 (Pin_5)
- net at U1.24 (PB5): now also J8.6 (Pin_6)
- net at U1.25 (PB6): now also J8.7 (Pin_7)
- net at U1.26 (PB7): now also J8.8 (Pin_8)
- net at U1.35 (PL0): now also J3.1 (Pin_1)
- net at U1.36 (PL1): now also J3.2 (Pin_2)
- net at U1.37 (PL2): now also J3.3 (Pin_3)
- net at U1.38 (PL3): now also J3.4 (Pin_4)
- net at U1.39 (PL4): now also J3.5 (Pin_5)
- net at U1.4 (PE2): now also J11.3 (Pin_3)
- net at U1.40 (PL5): now also J3.6 (Pin_6)
- net at U1.41 (PL6): now also J3.7 (Pin_7)
- net at U1.42 (PL7): now also J3.8 (Pin_8)
- net at U1.43 (PD0): now also J10.1 (Pin_1)
- net at U1.44 (PD1): now also J10.2 (Pin_2)
- net at U1.45 (PD2): now also J10.3 (Pin_3)
- net at U1.46 (PD3): now also J10.4 (Pin_4)
- net at U1.47 (PD4): now also J10.5 (Pin_5)
- net at U1.48 (PD5): now also J10.6 (Pin_6)
- net at U1.49 (PD6): now also J10.7 (Pin_7)
- net at U1.5 (PE3): now also J11.4 (Pin_4)
- net at U1.50 (PD7): now also J10.8 (Pin_8)
- net PG0: now reaches U1.51 (PG0)
- net PG1: now reaches U1.52 (PG1)
- net at U1.53 (PC0): now also J9.1 (Pin_1)
- net at U1.54 (PC1): now also J9.2 (Pin_2)
- net at U1.55 (PC2): now also J9.3 (Pin_3)
- net at U1.56 (PC3): now also J9.4 (Pin_4)
- net at U1.57 (PC4): now also J9.5 (Pin_5)
- net at U1.58 (PC5): now also J9.6 (Pin_6)
- net at U1.59 (PC6): now also J9.7 (Pin_7)
- net at U1.6 (PE4): now also J11.5 (Pin_5)
- net at U1.60 (PC7): now also J9.8 (Pin_8)
- net at U1.63 (PJ0): now also J5.1 (Pin_1)
- net at U1.64 (PJ1): now also J5.2 (Pin_2)
- net at U1.65 (PJ2): now also J5.3 (Pin_3)
- net at U1.66 (PJ3): now also J5.4 (Pin_4)
- net at U1.67 (PJ4): now also J5.5 (Pin_5)
- net at U1.68 (PJ5): now also J5.6 (Pin_6)
- net at U1.69 (PJ6): now also J5.7 (Pin_7)
- net at U1.7 (PE5): now also J11.6 (Pin_6)
- net at U1.71 (PA7): now also J7.8 (Pin_8)
- net at U1.72 (PA6): now also J7.7 (Pin_7)
- net at U1.73 (PA5): now also J7.6 (Pin_6)
- net at U1.74 (PA4): now also J7.5 (Pin_5)
- net at U1.75 (PA3): now also J7.4 (Pin_4)
- net at U1.76 (PA2): now also J7.3 (Pin_3)
- net at U1.77 (PA1): now also J7.2 (Pin_2)
- net at U1.78 (PA0): now also J7.1 (Pin_1)
- net at U1.79 (PJ7): now also J5.8 (Pin_8)
- net at U1.8 (PE6): now also J11.7 (Pin_7)
- net at U1.82 (PK7): now also J4.8 (Pin_8)
- net at U1.83 (PK6): now also J4.7 (Pin_7)
- net at U1.84 (PK5): now also J4.6 (Pin_6)
- net at U1.85 (PK4): now also J4.5 (Pin_5)
- net at U1.86 (PK3): now also J4.4 (Pin_4)
- net at U1.87 (PK2): now also J4.3 (Pin_3)
- net at U1.88 (PK1): now also J4.2 (Pin_2)
- net at U1.89 (PK0): now also J4.1 (Pin_1)
- net at U1.9 (PE7): now also J11.8 (Pin_8)
- net at U1.90 (PF7): now also J12.8 (Pin_8)
- net at U1.91 (PF6): now also J12.7 (Pin_7)
- net at U1.92 (PF5): now also J12.6 (Pin_6)
- net at U1.93 (PF4): now also J12.5 (Pin_5)
- net at U1.94 (PF3): now also J12.4 (Pin_4)
- net at U1.95 (PF2): now also J12.3 (Pin_3)
- net at U1.96 (PF1): now also J12.2 (Pin_2)
- net at U1.97 (PF0): now also J12.1 (Pin_1)
- new net: D2.2 (A), R9.1
- new net: D1.2 (A), R7.1
Other:
- moved on the sheet: J1, R3, R4, U2

Commit message: Almost done?
Parts:
- added JP1: IO0_JMP, Connector_PinHeader_2.54mm:PinHeader_1x02_P2.54mm_Vertical, symbol Jumper:Jumper_2_Open
- added JP2: RST_JMP, Connector_PinHeader_2.54mm:PinHeader_1x02_P2.54mm_Vertical, symbol Jumper:Jumper_2_Open
- added R5, R6: 10k, Resistor_SMD:R_0201_0603Metric, symbol Device:R
- D1: value LED -> FUN_LED_YEL
- D2: value LED_PWR -> LED_PWR_GRN
Connections:
- net +3V3: now also R5.1, R6.1; no longer J2.3 (Pin_3), J2.4 (Pin_4)
- net +5V: now also J14.1 (Pin_1); no longer J14.2 (Pin_2)
- net GND: now also J14.2 (Pin_2), JP1.2 (B), JP2.2 (B); no longer J14.1 (Pin_1)
- new net ESP_IO0: J2.3 (Pin_3), JP1.1 (A), R5.2
- new net ESP_RST: J2.4 (Pin_4), JP2.1 (A), R6.2
Other:
- note added: "3.3v voltage divider"
- note removed: "Step down voltage going to ESP8266 from 5V to 3.3V \nTechnically works without, but probably better for longevity"
- moved on the sheet: J14, R3, R4
