File: pcb_design/pcb_design.sch (KiCad schematic (older format))
At the start: 36 parts, among them J1 PWR_IN, J10 PD, J11 PE, J12 PF, J13 ICSP, J14 PWR_OUT, J2 ESP8266_CONN, J3 PL, J4 PK, J5 PJ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

Commit message: Add DS3231 RTC header
Parts:
- added J15: Conn_01x04, Connector_PinSocket_2.54mm:PinSocket_1x04_P2.54mm_Vertical, symbol Connector_Generic:Conn_01x04
Connections:
- net +5V: now also J15.3 (Pin_3)
- net GND: now also J15.4 (Pin_4)
- net SCL: now reaches J10.1 (Pin_1), U1.43 (PD0)
- net SCL: now also J15.1 (Pin_1)
- net SDA: now reaches J10.2 (Pin_2), U1.44 (PD1)
- net SDA: now also J15.2 (Pin_2)
Changed lines of the file:
@@
 	4350 4600 3800 4600
 Wire Wire Line
-	3800 4500 4350 4500
-Wire Wire Line
-	4350 4400 3800 4400
+	3800 4500 4150 4500
+Wire Wire Line
+	4350 4400 3850 4400
 Wire Wire Line
 	4350 4100 3800 4100
@@
 Wire Wire Line
 	1100 6700 1300 6700
+Text Label 4150 4300 0    50   ~ 0
+SDA
+Text Label 3850 4300 0    50   ~ 0
+SCL
+Wire Wire Line
+	3850 4400 3850 4300
+Connection ~ 3850 4400
+Wire Wire Line
+	3850 4400 3800 4400
+Wire Wire Line
+	4150 4300 4150 4500
+Connection ~ 4150 4500
+Wire Wire Line
+	4150 4500 4350 4500
+$Comp
+L Connector_Generic:Conn_01x04 J15
+U 1 1 607E0A85
+P 6100 5250
+F 0 "J15" H 6180 5242 50  0000 L CNN
+F 1 "Conn_01x04" H 6180 5151 50  0000 L CNN
+F 2 "Connector_PinSocket_2.54mm:PinSocket_1x04_P2.54mm_Vertical" H 6100 5250 50  0001 C CNN
+F 3 "~" H 6100 5250 50  0001 C CNN
+	1    6100 5250
+	1    0    0    -1
+$EndComp
+Text Label 5700 5250 2    50   ~ 0
+SDA
+Text Label 5700 5150 2    50   ~ 0
+SCL
+$Comp
+L power:+5V #PWR0127
+U 1 1 607E56A4
+P 5700 5350
+F 0 "#PWR0127" H 5700 5200 50  0001 C CNN
+F 1 "+5V" V 5715 5478 50  0000 L CNN
+F 2 "" H 5700 5350 50  0001 C CNN
+F 3 "" H 5700 5350 50  0001 C CNN
+	1    5700 5350
+	0    -1   -1   0
+$EndComp
+$Comp
+L power:GND #PWR0128
+U 1 1 607E6049
+P 5700 5450
+F 0 "#PWR0128" H 5700 5200 50  0001 C CNN
+F 1 "GND" V 5705 5322 50  0000 R CNN
+F 2 "" H 5700 5450 50  0001 C CNN
+F 3 "" H 5700 5450 50  0001 C CNN
+	1    5700 5450
+	0    1    1    0
+$EndComp
+Wire Wire Line
+	5700 5150 5900 5150
+Wire Wire Line
+	5900 5250 5700 5250
+Wire Wire Line
+	5700 5350 5900 5350
+Wire Wire Line
+	5900 5450 5700 5450
 $EndSCHEMATC

Commit message: Use correctly sized crystal, more changes
Parts:
- Clk1: footprint Crystal:Crystal_HC52-8mm_Vertical -> Crystal:Crystal_HC49-4H_Vertical
Changed lines of the file:
@@
 F 0 "Clk1" V 1554 2131 50  0000 L CNN
 F 1 "16Mhz" V 1645 2131 50  0000 L CNN
-F 2 "Crystal:Crystal_HC52-8mm_Vertical" H 1600 2000 50  0001 C CNN
+F 2 "Crystal:Crystal_HC49-4H_Vertical" H 1600 2000 50  0001 C CNN
 F 3 "~" H 1600 2000 50  0001 C CNN
 	1    1600 2000
