File: pcb_design/pcb_design.sch (KiCad schematic (older format))
At the start: 37 parts, among them J1 PWR_IN, J10 PD, J11 PE, J12 PF, J13 ICSP, J14 PWR_OUT, J15 Conn_01x04, J2 ESP8266_CONN, J3 PL, J4 PK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

Commit message: 0603EU -> 0603US
Parts:
- C1, C2, C3, C4, C5: footprint Capacitor_SMD:C_0201_0603Metric -> Capacitor_SMD:C_0603_1608Metric
- Clk1: footprint Crystal:Crystal_HC52-8mm_Vertical -> Crystal:Crystal_HC49-4H_Vertical
- D1, D2: footprint LED_SMD:LED_0201_0603Metric -> LED_SMD:LED_0603_1608Metric
- R1, R2, R3, R4, R5, R6, R7, R8, R9: footprint Resistor_SMD:R_0201_0603Metric -> Resistor_SMD:R_0603_1608Metric
Changed lines of the file:
@@
 F 0 "Clk1" V 1554 2131 50  0000 L CNN
 F 1 "16Mhz" V 1645 2131 50  0000 L CNN
-F 2 "Crystal:Crystal_HC52-8mm_Vertical" H 1600 2000 50  0001 C CNN
+F 2 "Crystal:Crystal_HC49-4H_Vertical" H 1600 2000 50  0001 C CNN
 F 3 "~" H 1600 2000 50  0001 C CNN
 	1    1600 2000
@@
 F 0 "R1" H 950 1950 50  0000 L CNN
 F 1 "1M" V 900 1950 50  0000 L CNN
-F 2 "Resistor_SMD:R_0201_0603Metric" V 830 2000 50  0001 C CNN
+F 2 "Resistor_SMD:R_0603_1608Metric" V 830 2000 50  0001 C CNN
 F 3 "~" H 900 2000 50  0001 C CNN
 	1    900  2000
@@
 F 0 "R2" V 2050 2150 50  0000 C CNN
 F 1 "27" V 1950 2150 50  0000 C CNN
-F 2 "Resistor_SMD:R_0201_0603Metric" V 1880 2150 50  0001 C CNN
+F 2 "Resistor_SMD:R_0603_1608Metric" V 1880 2150 50  0001 C CNN
 F 3 "~" H 1950 2150 50  0001 C CNN
 	1    1950 2150
@@
 F 0 "C1" V 1150 1850 50  0000 C CNN
 F 1 "22pF" V 1250 1850 50  0000 C CNN
-F 2 "Capacitor_SMD:C_0201_0603Metric" H 1350 1850 50  0001 C CNN
+F 2 "Capacitor_SMD:C_0603_1608Metric" H 1350 1850 50  0001 C CNN
 F 3 "~" H 1350 1850 50  0001 C CNN
 	1    1350 1850
@@
 F 0 "C2" V 1550 2150 50  0000 C CNN
 F 1 "22pF" V 1450 2150 50  0000 C CNN
-F 2 "Capacitor_SMD:C_0201_0603Metric" H 1350 2150 50  0001 C CNN
+F 2 "Capacitor_SMD:C_0603_1608Metric" H 1350 2150 50  0001 C CNN
 F 3 "~" H 1350 2150 50  0001 C CNN
 	1    1350 2150
@@
 F 0 "R3" V 5993 4250 50  0000 C CNN
 F 1 "10K" V 6084 4250 50  0000 C CNN
-F 2 "Resistor_SMD:R_0201_0603Metric" V 6130 4250 50  0001 C CNN
+F 2 "Resistor_SMD:R_0603_1608Metric" V 6130 4250 50  0001 C CNN
 F 3 "~" H 6200 4250 50  0001 C CNN
 	1    6200 4250
@@
 F 0 "R4" V 5693 4250 50  0000 C CNN
 F 1 "20K" V 5784 4250 50  0000 C CNN
-F 2 "Resistor_SMD:R_0201_0603Metric" V 5830 4250 50  0001 C CNN
+F 2 "Resistor_SMD:R_0603_1608Metric" V 5830 4250 50  0001 C CNN
 F 3 "~" H 5900 4250 50  0001 C CNN
 	1    5900 4250
@@
 F 0 "C3" H 3415 1296 50  0000 L CNN
 F 1 "100nF" H 3415 1205 50  0000 L CNN
-F 2 "Capacitor_SMD:C_0201_0603Metric" H 3338 1100 50  0001 C CNN
+F 2 "Capacitor_SMD:C_0603_1608Metric" H 3338 1100 50  0001 C CNN
 F 3 "~" H 3300 1250 50  0001 C CNN
 	1    3300 1250
@@
 F 0 "C4" H 3865 1296 50  0000 L CNN
 F 1 "100nF" H 3865 1205 50  0000 L CNN
-F 2 "Capacitor_SMD:C_0201_0603Metric" H 3788 1100 50  0001 C CNN
+F 2 "Capacitor_SMD:C_0603_1608Metric" H 3788 1100 50  0001 C CNN
 F 3 "~" H 3750 1250 50  0001 C CNN
 	1    3750 1250
@@
 F 0 "C5" H 4315 1296 50  0000 L CNN
 F 1 "100nF" H 4315 1205 50  0000 L CNN
-F 2 "Capacitor_SMD:C_0201_0603Metric" H 4238 1100 50  0001 C CNN
+F 2 "Capacitor_SMD:C_0603_1608Metric" H 4238 1100 50  0001 C CNN
 F 3 "~" H 4200 1250 50  0001 C CNN
 	1    4200 1250
@@
 F 0 "R8" H 2170 1546 50  0000 L CNN
 F 1 "10K" H 2170 1455 50  0000 L CNN
-F 2 "Resistor_SMD:R_0201_0603Metric" V 2030 1500 50  0001 C CNN
+F 2 "Resistor_SMD:R_0603_1608Metric" V 2030 1500 50  0001 C CNN
 F 3 "~" H 2100 1500 50  0001 C CNN
 	1    2100 1500
@@
 F 0 "D2" H 6793 1117 50  0000 C CNN
 F 1 "LED_PWR_GRN" H 6793 1026 50  0000 C CNN
-F 2 "LED_SMD:LED_0201_0603Metric" H 6800 900 50  0001 C CNN
+F 2 "LED_SMD:LED_0603_1608Metric" H 6800 900 50  0001 C CNN
 F 3 "~" H 6800 900 50  0001 C CNN
 	1    6800 900
@@
 F 0 "R9" V 7457 900 50  0000 C CNN
 F 1 "1K" V 7366 900 50  0000 C CNN
-F 2 "Resistor_SMD:R_0201_0603Metric" V 7180 900 50  0001 C CNN
+F 2 "Resistor_SMD:R_0603_1608Metric" V 7180 900 50  0001 C CNN
 F 3 "~" H 7250 900 50  0001 C CNN
 	1    7250 900
@@
 F 0 "D1" H 1443 6917 50  0000 C CNN
 F 1 "FUN_LED_YEL" H 1443 6826 50  0000 C CNN
-F 2 "LED_SMD:LED_0201_0603Metric" H 1450 6700 50  0001 C CNN
+F 2 "LED_SMD:LED_0603_1608Metric" H 1450 6700 50  0001 C CNN
 F 3 "~" H 1450 6700 50  0001 C CNN
 	1    1450 6700
@@
 F 0 "R7" V 2107 6700 50  0000 C CNN
 F 1 "1K" V 2016 6700 50  0000 C CNN
-F 2 "Resistor_SMD:R_0201_0603Metric" V 1830 6700 50  0001 C CNN
+F 2 "Resistor_SMD:R_0603_1608Metric" V 1830 6700 50  0001 C CNN
 F 3 "~" H 1900 6700 50  0001 C CNN
 	1    1900 6700
@@
 F 0 "R5" V 7200 3800 50  0000 C CNN
 F 1 "10k" V 7300 3800 50  0000 C CNN
-F 2 "Resistor_SMD:R_0201_0603Metric" V 7230 3800 50  0001 C CNN
+F 2 "Resistor_SMD:R_0603_1608Metric" V 7230 3800 50  0001 C CNN
 F 3 "~" H 7300 3800 50  0001 C CNN
 	1    7300 3800
@@
 F 0 "R6" V 7200 4350 50  0000 C CNN
 F 1 "10k" V 7300 4350 50  0000 C CNN
-F 2 "Resistor_SMD:R_0201_0603Metric" V 7230 4350 50  0001 C CNN
+F 2 "Resistor_SMD:R_0603_1608Metric" V 7230 4350 50  0001 C CNN
 F 3 "~" H 7300 4350 50  0001 C CNN
 	1    7300 4350
